Commit message: AUV now teleoperable

File: remaro_auv_description/urdf/base.xacro (robot description, xacro)
@@ -24,14 +24,11 @@
       <!-- Rigid body description of the base link -->
       <link name="${namespace}/base_link">
-        <!--
-          Be careful to setup the coefficients for the inertial tensor,
-          otherwise your model will become unstable on Gazebo
-        -->
+        <!-- Assuming uniform solid cylinder -->
         <inertial>
           <mass value="${remaro_auv_mass}" />
           <origin xyz="${remaro_auv_cog}" rpy="0 0 0"/>
-          <inertia ixx="${0.50*remaro_auv_mass*remaro_auv_radius*remaro_auv_radius}" ixy="0" ixz="0"
-                   iyy="${0.25*remaro_auv_mass*remaro_auv_radius*remaro_auv_radius + 0.083*remaro_auv_mass*remaro_auv_length*remaro_auv_length}" iyz="0"
-                   izz="${0.25*remaro_auv_mass*remaro_auv_radius*remaro_auv_radius + 0.083*remaro_auv_mass*remaro_auv_length*remaro_auv_length}" />
+          <inertia ixx="${1/2*remaro_auv_mass*remaro_auv_radius*remaro_auv_radius}" ixy="0" ixz="0"
+                   iyy="${1/4*remaro_auv_mass*remaro_auv_radius*remaro_auv_radius + 1/12*remaro_auv_mass*remaro_auv_length*remaro_auv_length}" iyz="0"
+                   izz="${1/4*remaro_auv_mass*remaro_auv_radius*remaro_auv_radius + 1/12*remaro_auv_mass*remaro_auv_length*remaro_auv_length}" />
         </inertial>
         <visual>

File: remaro_auv_description/urdf/gazebo.xacro (robot description, xacro)
@@ -2,17 +2,21 @@
 <robot xmlns:xacro="http://www.ros.org/wiki/xacro">
   <!-- Vehicle's parameters (remember to enter the model parameters below) -->
-    <!-- Describing the dimensions of the vehicle's bounding box -->
-    <xacro:property name="remaro_auv_length" value="3.0"/>
-    <xacro:property name="remaro_auv_width"  value="0.5"/>
-    <xacro:property name="remaro_auv_height" value="0.5"/>
-    <xacro:property name="remaro_auv_radius" value="${0.5*remaro_auv_width}"/>
-    <!-- Center of gravity -->
-    <xacro:property name="remaro_auv_mass" value="3228"/>
+    <xacro:property name="remaro_auv_length" value="3.00"/>
+    <xacro:property name="remaro_auv_radius" value="-0.1"/>
+    <!-- Buoyancy info -->
+    <xacro:property name="remaro_auv_buoyancy_kg" value="2"/>
+    <xacro:property name="remaro_auv_rho"  value="1027.5"/>
+    <xacro:property name="remaro_auv_cob" value="0 0 0.2"/>
+    <!-- Volume approximated as cylinder with hemispherical ends -->
+    <xacro:property
+      name="remaro_auv_volume"
+      value="${1/3*pi*remaro_auv_radius*remaro_auv_radius*(3*remaro_auv_length-2*remaro_auv_radius)}"
+    />
+    <!-- Mass info -->
+    <xacro:property
+      name="remaro_auv_mass"
+      value="${remaro_auv_volume*remaro_auv_rho-remaro_auv_buoyancy_kg}"
+    />
     <xacro:property name="remaro_auv_cog"  value="0 0 0"/>
-    <!-- Center of buoyancy -->
-    <xacro:property name="remaro_auv_rho"  value="1028"/>
-    <xacro:property name="remaro_auv_cob" value="0 0 0.1"/>
-    <!-- Vehicle's actual volume (Gazebo cannot compute the volume out of the mesh) -->
-    <xacro:property name="remaro_auv_volume" value="3.14*remaro_auv_radius*remaro_auv_radius*remaro_auv_length"/>
     <xacro:macro name="remaro_auv_hydro_model" params="namespace">
       <!-- List of hydrodynamic models this robot's links -->
@@ -26,29 +30,24 @@
         This is a workaround the invalid bounding box given by Gazebo-->
         <box>
-          <width> ${remaro_auv_width} </width>
+          <width> ${remaro_auv_volume/(2*remaro_auv_length*remaro_auv_radius)} </width>
           <length>${remaro_auv_length}</length>
-          <height>${remaro_auv_height}</height>
+          <height>${2*remaro_auv_radius}</height>
         </box>
         <!-- Center of buoyancy -->
         <center_of_buoyancy>${remaro_auv_cob}</center_of_buoyancy>
-        <!-- 1) Fossen's equation of motion -->
+        <!-- Fossen's equation of motion; values interpolated from example AUVs-->
         <hydrodynamic_model>
           <type>fossen</type>
           <added_mass>
-             5    0    0    0    0    0
-             0  100    0    0    0    0
-             0    0   80    0    0    0
-             0    0    0    0.5  0    0
-             0    0    0    0   30    0
-             0    0    0    0    0   35
+             50     0     0     0     0     0
+              0   400     0     0     0     0
+              0     0   400     0     0     0
+              0     0     0     0     0     0
+              0     0     0     0   400     0
+              0     0     0     0     0   400
           </added_mass>
-          <linear_damping_forward_speed>
-           -10    0    0    0    0    0
-             0 -180    0    0    0  180
-             0    0 -120    0 -120    0
-             0    0    0  -15    0    0
-             0    0   45    0  -25    0
-             0  -35    0    0    0  -35
-          </linear_damping_forward_speed>
+          <linear_damping>-30 -600 -400 -30 -100 -100</linear_damping>
+          <linear_damping_forward_speed>-30 -600 -400 -30 -100 -100</linear_damping_forward_speed>
+          <quadratic_damping>0 0 0 0 0 0</quadratic_damping>
         </hydrodynamic_model>
       </link>

File: remaro_auv_description/urdf/snippets.xacro (robot description, xacro)
@@ -49,10 +49,10 @@
         <gain>1</gain>
         <!-- Maximum allowed input value for the input signal for thruster unit -->
-        <clampMax>-3000</clampMax>
+        <clampMax>-100</clampMax>
         <!-- Minimum allowed value for the input signal for thruster unit -->
-        <clampMin>3000</clampMin>
+        <clampMin>100</clampMin>
         <!-- Minimum and maximum thrust force output allowed -->
-        <thrustMin>-50</thrustMin>
-        <thrustMax>50</thrustMax>
+        <thrustMin>-100</thrustMin>
+        <thrustMax>100</thrustMax>
         <!--
         Value from 0 to 1 to set the efficiency of the output thrust force
@@ -69,9 +69,9 @@
         <dynamics>
           <type>FirstOrder</type>
-          <timeConstant>0.05</timeConstant>
+          <timeConstant>0.08</timeConstant>
         </dynamics>
         <conversion>
           <type>Basic</type>
-          <rotorConstant>0.0002</rotorConstant>
+          <rotorConstant>0.00008</rotorConstant>
         </conversion>
       </plugin>
@@ -86,7 +86,7 @@
   <!-- Fin properties -->
   <xacro:property name="fin_area" value="0.04"/>
-  <xacro:property name="fin_rho"  value="1028"/>
-  <xacro:property name="fin_lift_coefficient" value="3.0"/>
-  <xacro:property name="fin_drag_coefficient" value="2.0"/>
+  <xacro:property name="fin_rho"  value="1027.5"/>
+  <xacro:property name="fin_lift_coefficient" value="1.0"/>
+  <xacro:property name="fin_drag_coefficient" value="0.1"/>
   <xacro:macro name="fin_macro" params="namespace fin_id *origin mesh_filename">
       <xacro:fin_quadratic_macro
@@ -94,6 +94,6 @@
         parent_link="${namespace}/base_link"
         fin_id="${fin_id}"
-        min_joint_limit="${-75.0*d2r}"
-        max_joint_limit="${ 75.0*d2r}"
+        min_joint_limit="${-75*d2r}"
+        max_joint_limit="${ 75*d2r}"
         mesh_filename="${mesh_filename}"
         fin_dynamics_time_constant="0.2"
